File: Hardware/PCB V3 - Leandro/PCB V3 - Leandro/PCB V3 - Leandro.kicad_sch (KiCad schematic)
At the start: 15 parts, among them J1 Bateria (-), J10 MOTOR_DER, J2 Bateria (+), J3 Sensor TATAMI FD, J4 SWITCH, J5 Sensor TATAMI FI, J6 STEP_DOWN, J7 IR_FD, J8 IR_FI, J9 MOTOR_IZQ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

Commit message: termine la placa hay que ver que dice bustos
Parts:
- J1: value Bateria (-) -> (none)
- J2: value Bateria (+) -> (none)
Connections:
- net IR_D is gone; now on net ESTRATEGIA: U1.5 (IO35)
- net +5V: now also SW1.1, SW2.1
- net BUZZER: now also U1.30 (IO23); no longer U1.29 (IO22)
- net ESTRATEGIA: no longer U1.4 (IO34)
- net GND: no longer SW1.1, SW2.1
- net M1A: now also U1.26 (IO21); no longer U1.24 (IO18)
- net M1B: now also U1.29 (IO22); no longer U1.30 (IO23)
- net M2A: now also U1.24 (IO18); no longer U1.26 (IO21)
- net START: now also U1.4 (IO34); no longer U1.3 (SENSOR_VN)
- no-connect marks 11 -> 13
Other:
- note added: "BUZZER"
- note added: "Salidas para Motores"
- moved on the sheet: BZ1, J10, J3, J5, J6, J7, J8, J9, SW1, SW2

Commit message: falta la correccion de Bustos y diseñar el svg
Parts:
- removed J2: (no value), EESTN5:BORNERA2_AZUL, symbol EESTN5:TB_1X2
- removed J4: SWITCH, EESTN5:SW_SPDT_TH_Vertical, symbol EESTN5:Conn_01X03
- J1: value (none) -> Bateria (+)
Connections:
- net GND: now also J1.1
- net Vstep: now also J1.2
- removed net VBAT: J1.1, J1.2
Other:
- moved on the sheet: J1, J6

Commit message: placa para fabricar ya
Parts:
- added H1, H2: Mounting_Hole, EESTN5:pad_3mm, symbol EESTN5:Mounting_Hole
- added J2: IR_COSTADO, EESTN5:Pin_Strip_3, symbol EESTN5:Conn_01X03
Connections:
- net IR_I is gone; now on net IR_FI: U1.8 (IO25)
- net +5V: now also J2.2 (P2)
- net GND: now also J2.3 (P3)
- net IR_FD: now also U1.7 (IO33); no longer U1.6 (IO32)
- net IR_FI: no longer U1.7 (IO33)
- new net IR_COSTADO: J2.1 (P1), U1.6 (IO32)
Other:
- note added: "AGUJEROS DE SUJECION"
- moved on the sheet: Display1

Commit message: cambios de sch
Connections:
- net IR_COSTADO: now also U1.8 (IO25); no longer U1.6 (IO32)
- net IR_FI: now also U1.6 (IO32); no longer U1.8 (IO25)
- net M1A renamed M1A_PWM
- net M1B renamed M1B_DIR
- net M2A renamed M2A_PWM
- net M2B renamed M2B_DIR
Changed lines of the file:
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@@
     (effects (font (size 1.524 1.524)) (justify left bottom))
   )
-  (label "M1A" (at 144.272 35.56 0)
+  (label "M1A_PWM" (at 144.272 35.56 0)
     (effects (font (size 1.524 1.524)) (justify left bottom))
   )
@@
     (effects (font (size 1.524 1.524)) (justify left bottom))
   )
-  (label "IR_FI" (at 101.6 43.18 180)
+  (label "IR_FI" (at 101.6 38.1 180)
     (effects (font (size 1.524 1.524)) (justify right bottom))
   )
@@
     (effects (font (size 1.27 1.27)) (justify left bottom))
   )
-  (label "M1B" (at 144.526 27.94 0)
+  (label "M1B_DIR" (at 144.526 27.94 0)
     (effects (font (size 1.524 1.524)) (justify left bottom))
   )
@@
     (effects (font (size 1.524 1.524)) (justify right bottom))
   )
-  (label "M2A" (at 257.048 40.386 180)
+  (label "M2A_PWM" (at 257.048 40.386 180)
     (effects (font (size 1.524 1.524)) (justify right bottom))
   )
@@
     (effects (font (size 1.27 1.27)) (justify right bottom))
   )
-  (label "M2B" (at 257.048 45.466 180)
+  (label "M2B_DIR" (at 257.048 45.466 180)
     (effects (font (size 1.524 1.524)) (justify right bottom))
   )
-  (label "IR_COSTADO" (at 101.6 38.1 180)
+  (label "IR_COSTADO" (at 101.6 43.18 180)
     (effects (font (size 1.27 1.27)) (justify right bottom))
   )
@@
     (effects (font (size 1.27 1.27)) (justify right bottom))
   )
-  (label "M2B" (at 144.272 38.1 0)
+  (label "M2B_DIR" (at 144.272 38.1 0)
     (effects (font (size 1.524 1.524)) (justify left bottom))
   )
-  (label "M1A" (at 217.17 40.132 180)
+  (label "M1A_PWM" (at 217.17 40.132 180)
     (effects (font (size 1.524 1.524)) (justify right bottom))
   )
@@
     (effects (font (size 1.524 1.524)) (justify right bottom))
   )
-  (label "M2A" (at 144.272 40.64 0)
+  (label "M2A_PWM" (at 144.272 40.64 0)
     (effects (font (size 1.524 1.524)) (justify left bottom))
   )
@@
     (effects (font (size 1.524 1.524)) (justify right bottom))
   )
-  (label "M1B" (at 217.17 45.212 180)
+  (label "M1B_DIR" (at 217.17 45.212 180)
     (effects (font (size 1.524 1.524)) (justify right bottom))
   )
